File: boards/breakout.sch (EAGLE design)
At the start: 28 parts, among them Q2 BC846BSMD, Q4 BC846BSMD

Commit message: Made some minor changes
Connections:
- net GND: now also S7.3
Changed lines of the file:
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@@
 <wire x1="381" y1="124.46" x2="381" y2="83.82" width="0.1524" layer="91"/>
 <junction x="381" y="124.46"/>
-<wire x1="381" y1="208.28" x2="381" y2="124.46" width="0.1524" layer="91"/>
+<wire x1="381" y1="208.28" x2="381" y2="177.8" width="0.1524" layer="91"/>
 <pinref part="S2" gate="A" pin="3"/>
+<wire x1="381" y1="177.8" x2="381" y2="124.46" width="0.1524" layer="91"/>
 <wire x1="314.96" y1="223.52" x2="322.58" y2="223.52" width="0.1524" layer="91"/>
 <wire x1="314.96" y1="210.82" x2="314.96" y2="223.52" width="0.1524" layer="91"/>
@@
 <wire x1="304.8" y1="83.82" x2="307.34" y2="83.82" width="0.1524" layer="91"/>
 <wire x1="307.34" y1="83.82" x2="307.34" y2="96.52" width="0.1524" layer="91"/>
+<wire x1="381" y1="177.8" x2="360.68" y2="177.8" width="0.1524" layer="91"/>
+<wire x1="360.68" y1="177.8" x2="360.68" y2="182.88" width="0.1524" layer="91"/>
+<pinref part="S7" gate="A" pin="3"/>
+<wire x1="360.68" y1="182.88" x2="370.84" y2="182.88" width="0.1524" layer="91"/>
 </segment>
 <segment>
